File: ESP32-Breakout.kicad_sch (KiCad schematic)
At the start: 3 parts, among them J101 Conn_01x19, J102 Conn_01x19, U101 ESP32-DEVKITC-32D

Commit message: Production
Parts:
- J101, J102, U101: now left out of the parts list
Changed lines of the file:
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@@
   )
   (symbol (lib_id "Connector_Generic:Conn_01x19") (at 170.815 94.615 0) (unit 1)
-    (in_bom yes) (on_board yes)
+    (in_bom no) (on_board yes)
     (property "Reference" "J102" (id 0) (at 177.165 92.075 0)
       (effects (font (size 1.27 1.27)) (justify left))
@@
   )
   (symbol (lib_id "Connector_Generic:Conn_01x19") (at 110.49 94.615 0) (mirror y) (unit 1)
-    (in_bom yes) (on_board yes)
+    (in_bom no) (on_board yes)
     (property "Reference" "J101" (id 0) (at 102.235 92.075 0))
     (property "Value" "Conn_01x19" (id 1) (at 102.235 94.615 0))
@@
   )
   (symbol (lib_id "MCU_Module:ESP32-DEVKITC-32D") (at 140.335 94.615 0) (unit 1)
-    (in_bom yes) (on_board yes) (fields_autoplaced)
+    (in_bom no) (on_board yes) (fields_autoplaced)
     (property "Reference" "U101" (id 0) (at 140.335 63.5 0))
     (property "Value" "ESP32-DEVKITC-32D" (id 1) (at 140.335 66.04 0))

Commit message: Added 3D stacking header
Parts:
- U101: footprint Module:MODULE_ESP32-DEVKITC-32D -> ESP32:MODULE_ESP32-DEVKITC-32D
Changed lines of the file:
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@@
     (property "Reference" "U101" (id 0) (at 140.335 63.5 0))
     (property "Value" "ESP32-DEVKITC-32D" (id 1) (at 140.335 66.04 0))
-    (property "Footprint" "Module:MODULE_ESP32-DEVKITC-32D" (id 2) (at 140.335 94.615 0)
+    (property "Footprint" "ESP32:MODULE_ESP32-DEVKITC-32D" (id 2) (at 140.335 94.615 0)
       (effects (font (size 1.27 1.27)) (justify bottom) hide)
     )
@@
     )
     (path "/d7debd12-f7b7-4fce-af13-ea37ff0fb5af"
-      (reference "U101") (unit 1) (value "ESP32-DEVKITC-32D") (footprint "Module:MODULE_ESP32-DEVKITC-32D")
+      (reference "U101") (unit 1) (value "ESP32-DEVKITC-32D") (footprint "ESP32:MODULE_ESP32-DEVKITC-32D")
     )
   )

Commit message: Names streamlined
Parts:
- U101: footprint ESP32:MODULE_ESP32-DEVKITC-32D -> ESP32:MODULE_ESP32-DEVKITC-32D_Stacking_header_TH
Changed lines of the file:
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@@
     (property "Reference" "U101" (id 0) (at 140.335 63.5 0))
     (property "Value" "ESP32-DEVKITC-32D" (id 1) (at 140.335 66.04 0))
-    (property "Footprint" "ESP32:MODULE_ESP32-DEVKITC-32D" (id 2) (at 140.335 94.615 0)
+    (property "Footprint" "ESP32:MODULE_ESP32-DEVKITC-32D_Stacking_header_TH" (id 2) (at 140.335 94.615 0)
       (effects (font (size 1.27 1.27)) (justify bottom) hide)
     )
@@
     )
     (path "/d7debd12-f7b7-4fce-af13-ea37ff0fb5af"
-      (reference "U101") (unit 1) (value "ESP32-DEVKITC-32D") (footprint "ESP32:MODULE_ESP32-DEVKITC-32D")
+      (reference "U101") (unit 1) (value "ESP32-DEVKITC-32D") (footprint "ESP32:MODULE_ESP32-DEVKITC-32D_Stacking_header_TH")
     )
   )

Commit message: Closed #1
Other:
- moved on the sheet: J102
Changed lines of the file:
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@@
   (title_block
     (title "ESP32 breakout board")
-    (date "2023-01-30")
-    (rev "1.0.0")
+    (date "2023-02-08")
+    (rev "1.1.0")
     (company "Resterampe Berlin")
     (comment 3 "https://creativecommons.org/licenses/by-nc/4.0")
@@
     (stroke (width 0) (type default) (color 0 0 0 0))
   )
-  (wire (pts (xy 160.655 84.455) (xy 165.735 84.455))
+  (wire (pts (xy 160.655 84.455) (xy 165.1 84.455))
     (stroke (width 0) (type default) (color 0 0 0 0))
   )
@@
     (stroke (width 0) (type default) (color 0 0 0 0))
   )
-  (wire (pts (xy 160.655 81.915) (xy 165.735 81.915))
+  (wire (pts (xy 160.655 81.915) (xy 165.1 81.915))
     (stroke (width 0) (type default) (color 0 0 0 0))
   )
@@
     (stroke (width 0) (type default) (color 0 0 0 0))
   )
-  (wire (pts (xy 160.655 104.775) (xy 165.735 104.775))
+  (wire (pts (xy 160.655 104.775) (xy 165.1 104.775))
     (stroke (width 0) (type default) (color 0 0 0 0))
   )
@@
     (stroke (width 0) (type default) (color 0 0 0 0))
   )
-  (wire (pts (xy 163.195 86.995) (xy 165.735 86.995))
+  (wire (pts (xy 163.195 86.995) (xy 165.1 86.995))
     (stroke (width 0) (type default) (color 0 0 0 0))
   )
@@
     (stroke (width 0) (type default) (color 0 0 0 0))
   )
-  (wire (pts (xy 160.655 92.075) (xy 165.735 92.075))
+  (wire (pts (xy 160.655 92.075) (xy 165.1 92.075))
     (stroke (width 0) (type default) (color 0 0 0 0))
   )
@@
     (stroke (width 0) (type default) (color 0 0 0 0))
   )
-  (wire (pts (xy 160.655 89.535) (xy 165.735 89.535))
-    (stroke (width 0) (type default) (color 0 0 0 0))
-  )
-  (wire (pts (xy 160.655 99.695) (xy 165.735 99.695))
+  (wire (pts (xy 160.655 89.535) (xy 165.1 89.535))
+    (stroke (width 0) (type default) (color 0 0 0 0))
+  )
+  (wire (pts (xy 160.655 99.695) (xy 165.1 99.695))
     (stroke (width 0) (type default) (color 0 0 0 0))
   )
@@
     (stroke (width 0) (type default) (color 0 0 0 0))
   )
-  (wire (pts (xy 160.655 114.935) (xy 165.735 114.935))
-    (stroke (width 0) (type default) (color 0 0 0 0))
-  )
-  (wire (pts (xy 160.655 109.855) (xy 165.735 109.855))
-    (stroke (width 0) (type default) (color 0 0 0 0))
-  )
-  (wire (pts (xy 160.655 112.395) (xy 165.735 112.395))
-    (stroke (width 0) (type default) (color 0 0 0 0))
-  )
-  (wire (pts (xy 160.655 117.475) (xy 165.735 117.475))
+  (wire (pts (xy 160.655 114.935) (xy 165.1 114.935))
+    (stroke (width 0) (type default) (color 0 0 0 0))
+  )
+  (wire (pts (xy 160.655 109.855) (xy 165.1 109.855))
+    (stroke (width 0) (type default) (color 0 0 0 0))
+  )
+  (wire (pts (xy 160.655 112.395) (xy 165.1 112.395))
+    (stroke (width 0) (type default) (color 0 0 0 0))
+  )
+  (wire (pts (xy 160.655 117.475) (xy 165.1 117.475))
     (stroke (width 0) (type default) (color 0 0 0 0))
   )
@@
     (stroke (width 0) (type default) (color 0 0 0 0))
   )
-  (wire (pts (xy 160.655 74.295) (xy 165.735 74.295))
-    (stroke (width 0) (type default) (color 0 0 0 0))
-  )
-  (wire (pts (xy 163.195 71.755) (xy 165.735 71.755))
-    (stroke (width 0) (type default) (color 0 0 0 0))
-  )
-  (wire (pts (xy 160.655 97.155) (xy 165.735 97.155))
-    (stroke (width 0) (type default) (color 0 0 0 0))
-  )
-  (wire (pts (xy 160.655 76.835) (xy 165.735 76.835))
+  (wire (pts (xy 160.655 74.295) (xy 165.1 74.295))
+    (stroke (width 0) (type default) (color 0 0 0 0))
+  )
+  (wire (pts (xy 163.195 71.755) (xy 165.1 71.755))
+    (stroke (width 0) (type default) (color 0 0 0 0))
+  )
+  (wire (pts (xy 160.655 97.155) (xy 165.1 97.155))
+    (stroke (width 0) (type default) (color 0 0 0 0))
+  )
+  (wire (pts (xy 160.655 76.835) (xy 165.1 76.835))
     (stroke (width 0) (type default) (color 0 0 0 0))
   )
@@
     (stroke (width 0) (type default) (color 0 0 0 0))
   )
-  (wire (pts (xy 160.655 102.235) (xy 165.735 102.235))
+  (wire (pts (xy 160.655 102.235) (xy 165.1 102.235))
     (stroke (width 0) (type default) (color 0 0 0 0))
   )
@@
     (stroke (width 0) (type default) (color 0 0 0 0))
   )
-  (wire (pts (xy 160.655 107.315) (xy 165.735 107.315))
-    (stroke (width 0) (type default) (color 0 0 0 0))
-  )
-  (wire (pts (xy 160.655 79.375) (xy 165.735 79.375))
+  (wire (pts (xy 160.655 107.315) (xy 165.1 107.315))
+    (stroke (width 0) (type default) (color 0 0 0 0))
+  )
+  (wire (pts (xy 160.655 79.375) (xy 165.1 79.375))
     (stroke (width 0) (type default) (color 0 0 0 0))
   )
@@
     (stroke (width 0) (type default) (color 0 0 0 0))
   )
-  (wire (pts (xy 160.655 94.615) (xy 165.735 94.615))
+  (wire (pts (xy 160.655 94.615) (xy 165.1 94.615))
     (stroke (width 0) (type default) (color 0 0 0 0))
   )
@@
     (pin "1")
   )
-  (symbol (lib_id "Connector_Generic:Conn_01x19") (at 170.815 94.615 0) (unit 1)
+  (symbol (lib_id "Connector_Generic:Conn_01x19") (at 170.18 94.615 0) (unit 1)
     (in_bom no) (on_board yes)
-    (property "Reference" "J102" (id 0) (at 177.165 92.075 0)
+    (property "Reference" "J102" (id 0) (at 176.53 92.075 0)
       (effects (font (size 1.27 1.27)) (justify left))
     )
-    (property "Value" "Conn_01x19" (id 1) (at 173.355 94.615 0)
+    (property "Value" "Conn_01x19" (id 1) (at 172.72 94.615 0)
       (effects (font (size 1.27 1.27)) (justify left))
     )
-    (property "Footprint" "Connector_PinHeader_2.54mm:PinHeader_1x19_P2.54mm_Vertical" (id 2) (at 170.815 94.615 0)
-      (effects (font (size 1.27 1.27)) hide)
-    )
-    (property "Datasheet" "~" (id 3) (at 170.815 94.615 0)
-      (effects (font (size 1.27 1.27)) hide)
-    )
+    (property "Footprint" "Connector_PinHeader_2.54mm:PinHeader_1x19_P2.54mm_Vertical" (id 2) (at 170.18 94.615 0)
+      (effects (font (size 1.27 1.27)) hide)
+    )
+    (property "Datasheet" "~" (id 3) (at 170.18 94.615 0)
+      (effects (font (size 1.27 1.27)) hide)
+    )
